File: PCB/OeMRFM69_USB.kicad_sch (KiCad schematic)
At the start: 23 parts, among them J1 AERIAL, J2 TYPE-C-31-M-12, U1 ATtiny1624-SS, U2 RFM69CW, U4 XC6206-3.3V, U5 CH340C

Commit message: Updated BOM
Parts:
- C1, C5: LCSCStockCode (none) -> C15850; PartNumber (none) -> CL21A106KAYNNNE
- C2, C3: LCSCStockCode (none) -> C49678; PartNumber (none) -> CC0805KRX7R9BB104
- C4: LCSCStockCode (none) -> C1779; PartNumber (none) -> CL21A475KAQNNNE
- D1: LCSCStockCode (none) -> C84256; PartNumber (none) -> NCD0805R1
- D3: PartNumber (none) -> BAT46W
- JP1, JP2: footprint Connector_PinSocket_2.54mm:PinSocket_1x02_P2.54mm_Vertical -> Connector_PinHeader_2.54mm:PinHeader_1x02_P2.54mm_Vertical; LCSCStockCode (none) -> C2833329; PartNumber (none) -> KH-A2541WV-2P
- R1: LCSCStockCode (none) -> C17414; PartNumber (none) -> 0805W8F1002T5E
- R2, R6, R7: LCSCStockCode (none) -> C17513; PartNumber (none) -> 0805W8F1001T5E
- R3: LCSCStockCode (none) -> C149504; PartNumber (none) -> 0805W8F1003T5E
- R4, R5: LCSCStockCode (none) -> C27834; PartNumber (none) -> 0805W8F5101T5E
- UPDI1: now left out of the parts list
Changed lines of the file:
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@@
   )
   (symbol (lib_id "Connector_Generic:Conn_01x03") (at 234.95 99.06 0) (unit 1)
-    (in_bom yes) (on_board yes) (dnp no)
+    (in_bom no) (on_board yes) (dnp no)
     (property "Reference" "UPDI1" (at 237.6932 91.9226 0)
       (effects (font (size 1.27 1.27)))
@@
       (effects (font (size 1.27 1.27)) hide)
     )
+    (property "LCSCStockCode" "C17414" (at 146.05 120.65 0)
+      (effects (font (size 1.27 1.27)) hide)
+    )
+    (property "PartNumber" "0805W8F1002T5E" (at 146.05 120.65 0)
+      (effects (font (size 1.27 1.27)) hide)
+    )
     (pin "1")
     (pin "2")
@@
       (effects (font (size 1.27 1.27)) hide)
     )
+    (property "LCSCStockCode" "C49678" (at 71.12 102.87 0)
+      (effects (font (size 1.27 1.27)) hide)
+    )
+    (property "PartNumber" "CC0805KRX7R9BB104" (at 71.12 102.87 0)
+      (effects (font (size 1.27 1.27)) hide)
+    )
     (pin "1")
     (pin "2")
@@
       (effects (font (size 1.27 1.27)) hide)
     )
+    (property "LCSCStockCode" "C17513" (at 147.32 162.56 0)
+      (effects (font (size 1.27 1.27)) hide)
+    )
+    (property "PartNumber" "0805W8F1001T5E" (at 147.32 162.56 0)
+      (effects (font (size 1.27 1.27)) hide)
+    )
     (pin "1")
     (pin "2")
@@
     )
     (property "Datasheet" "~" (at 274.32 38.1 0)
+      (effects (font (size 1.27 1.27)) hide)
+    )
+    (property "LCSCStockCode" "C49678" (at 274.32 38.1 0)
+      (effects (font (size 1.27 1.27)) hide)
+    )
+    (property "PartNumber" "CC0805KRX7R9BB104" (at 274.32 38.1 0)
       (effects (font (size 1.27 1.27)) hide)
     )
@@
       (effects (font (size 1.27 1.27)) hide)
     )
+    (property "LCSCStockCode" "C17513" (at 125.73 171.45 0)
+      (effects (font (size 1.27 1.27)) hide)
+    )
+    (property "PartNumber" "0805W8F1001T5E" (at 125.73 171.45 0)
+      (effects (font (size 1.27 1.27)) hide)
+    )
     (pin "1")
     (pin "2")
@@
       (effects (font (size 1.27 1.27)) hide)
     )
+    (property "PartNumber" "BAT46W" (at 134.62 171.45 0)
+      (effects (font (size 1.27 1.27)) hide)
+    )
     (pin "1")
     (pin "2")
@@
       (effects (font (size 1.27 1.27)) hide)
     )
+    (property "LCSCStockCode" "C17513" (at 255.27 107.95 0)
+      (effects (font (size 1.27 1.27)) hide)
+    )
+    (property "PartNumber" "0805W8F1001T5E" (at 255.27 107.95 0)
+      (effects (font (size 1.27 1.27)) hide)
+    )
     (pin "1")
     (pin "2")
@@
       (effects (font (size 1.27 1.27)) hide)
     )
+    (property "LCSCStockCode" "C149504" (at 116.84 99.06 0)
+      (effects (font (size 1.27 1.27)) hide)
+    )
+    (property "PartNumber" "0805W8F1003T5E" (at 116.84 99.06 0)
+      (effects (font (size 1.27 1.27)) hide)
+    )
     (pin "1")
     (pin "2")
@@
       (effects (font (size 1.27 1.27)) hide)
     )
-    (property "PartNumber" "" (at 130.81 44.45 0)
-      (effects (font (size 1.27 1.27)) hide)
-    )
-    (property "LCSCStockCode" "" (at 130.81 44.45 0)
+    (property "PartNumber" "CL21A475KAQNNNE" (at 130.81 44.45 0)
+      (effects (font (size 1.27 1.27)) hide)
+    )
+    (property "LCSCStockCode" "C1779" (at 130.81 44.45 0)
       (effects (font (size 1.27 1.27)) hide)
     )
@@
       (effects (font (size 1.27 1.27)) hide)
     )
+    (property "LCSCStockCode" "C84256" (at 255.27 118.11 0)
+      (effects (font (size 1.27 1.27)) hide)
+    )
+    (property "PartNumber" "NCD0805R1" (at 255.27 118.11 0)
+      (effects (font (size 1.27 1.27)) hide)
+    )
     (pin "1")
     (pin "2")
@@
       (effects (font (size 1.27 1.27)) hide)
     )
+    (property "LCSCStockCode" "C27834" (at 227.33 41.91 0)
+      (effects (font (size 1.27 1.27)) hide)
+    )
+    (property "PartNumber" "0805W8F5101T5E" (at 227.33 41.91 0)
+      (effects (font (size 1.27 1.27)) hide)
+    )
     (pin "1")
     (pin "2")
@@
       (effects (font (size 1.27 1.27)) hide)
     )
+    (property "LCSCStockCode" "C15850" (at 196.85 109.22 0)
+      (effects (font (size 1.27 1.27)) hide)
+    )
+    (property "PartNumber" "CL21A106KAYNNNE" (at 196.85 109.22 0)
+      (effects (font (size 1.27 1.27)) hide)
+    )
     (pin "1")
     (pin "2")
@@
       (effects (font (size 1.27 1.27)))
     )
-    (property "Footprint" "Connector_PinSocket_2.54mm:PinSocket_1x02_P2.54mm_Vertical" (at 114.3 171.45 0)
+    (property "Footprint" "Connector_PinHeader_2.54mm:PinHeader_1x02_P2.54mm_Vertical" (at 114.3 171.45 0)
       (effects (font (size 1.27 1.27)) hide)
     )
     (property "Datasheet" "~" (at 114.3 171.45 0)
+      (effects (font (size 1.27 1.27)) hide)
+    )
+    (property "LCSCStockCode" "C2833329" (at 114.3 171.45 0)
+      (effects (font (size 1.27 1.27)) hide)
+    )
+    (property "PartNumber" "KH-A2541WV-2P" (at 114.3 171.45 0)
       (effects (font (size 1.27 1.27)) hide)
     )
@@
       (effects (font (size 1.27 1.27)) hide)
     )
+    (property "LCSCStockCode" "C27834" (at 227.33 39.37 0)
+      (effects (font (size 1.27 1.27)) hide)
+    )
+    (property "PartNumber" "0805W8F5101T5E" (at 227.33 39.37 0)
+      (effects (font (size 1.27 1.27)) hide)
+    )
     (pin "1")
     (pin "2")
@@
       (effects (font (size 1.27 1.27)) hide)
     )
-    (property "PartNumber" "" (at 158.75 41.91 0)
-      (effects (font (size 1.27 1.27)) hide)
-    )
-    (property "LCSCStockCode" "" (at 158.75 41.91 0)
+    (property "PartNumber" "CL21A106KAYNNNE" (at 158.75 41.91 0)
+      (effects (font (size 1.27 1.27)) hide)
+    )
+    (property "LCSCStockCode" "C15850" (at 158.75 41.91 0)
       (effects (font (size 1.27 1.27)) hide)
     )
@@
       (effects (font (size 1.27 1.27)))
     )
-    (property "Footprint" "Connector_PinSocket_2.54mm:PinSocket_1x02_P2.54mm_Vertical" (at 114.3 162.56 0)
+    (property "Footprint" "Connector_PinHeader_2.54mm:PinHeader_1x02_P2.54mm_Vertical" (at 114.3 162.56 0)
       (effects (font (size 1.27 1.27)) hide)
     )
@@
       (effects (font (size 1.27 1.27)) hide)
     )
+    (property "LCSCStockCode" "C2833329" (at 114.3 162.56 0)
+      (effects (font (size 1.27 1.27)) hide)
+    )
+    (property "PartNumber" "KH-A2541WV-2P" (at 114.3 162.56 0)
+      (effects (font (size 1.27 1.27)) hide)
+    )
